Commit message: feat: resolve UGV mobility in Gazebo with Direct-Proxy architecture and sensor re-integration

File: install/rover_description/share/rover_description/urdf/rover.urdf.xacro (robot description, xacro)
@@ -1,127 +1 @@
-<?xml version="1.0"?>
-<robot name="ugv" xmlns:xacro="http://www.ros.org/wiki/xacro">
-  <!-- ================= BASE FRAME (AXLE FRAME) ================= -->
-  <link name="base_link"/>
-  <!-- ================= CHASSIS ================= -->
-  <link name="chassis_link">
-    <inertial>
-      <mass value="450.0"/>
-      <origin xyz="0 0 0.2"/>
-      <inertia ixx="60" iyy="42" izz="91.5"
-               ixy="0" ixz="0" iyz="0"/>
-    </inertial>
-    <visual>
-      <origin xyz="0 0 0.2"/>
-      <geometry>
-        <box size="1.0 1.2 0.4"/>
-      </geometry>
-    </visual>
-    <collision>
-      <origin xyz="0 0 0.2"/>
-      <geometry>
-        <box size="1.0 1.2 0.4"/>
-      </geometry>
-    </collision>
-  </link>
-  <joint name="base_to_chassis" type="fixed">
-    <parent link="base_link"/>
-    <child link="chassis_link"/>
-    <origin xyz="0 0 -0.092"/>
-  </joint>
-  <!-- ================= WHEEL MACRO ================= -->
-  <xacro:macro name="wheel" params="name x y">
-    <link name="${name}">
-      <visual>
-        <origin rpy="1.5707 0 0"/>
-        <geometry>
-          <cylinder radius="0.292" length="0.12"/>
-        </geometry>
-      </visual>
-      <collision>
-        <origin rpy="1.5707 0 0"/>
-        <geometry>
-          <cylinder radius="0.292" length="0.12"/>
-        </geometry>
-      </collision>
-      <inertial>
-        <mass value="15"/>
-        <origin xyz="0 0 0"/>
-        <inertia ixx="0.34" iyy="0.34" izz="0.64"
-                 ixy="0" ixz="0" iyz="0"/>
-      </inertial>
-    </link>
-    <joint name="${name}_joint" type="continuous">
-      <parent link="base_link"/>
-      <child link="${name}"/>
-      <origin xyz="${x} ${y} 0"/>
-      <axis xyz="0 1 0"/>
-    </joint>
-    <gazebo reference="${name}">
-      <mu1>3.0</mu1>
-      <mu2>3.0</mu2>
-      <kp>100000</kp>
-      <kd>10</kd>
-    </gazebo>
-  </xacro:macro>
-  <!-- ================= WHEELS ================= -->
-  <xacro:wheel name="front_left_wheel"  x="0.4"  y="0.675"/>
-  <xacro:wheel name="front_right_wheel" x="0.4"  y="-0.675"/>
-  <xacro:wheel name="rear_left_wheel"   x="-0.4" y="0.675"/>
-  <xacro:wheel name="rear_right_wheel"  x="-0.4" y="-0.675"/>
-  <!-- ================= SENSORS ================= -->
-  <link name="lidar_link"/>
-  <joint name="lidar_joint" type="fixed">
-    <parent link="chassis_link"/>
-    <child link="lidar_link"/>
-    <origin xyz="0.2 0 0.4"/>
-  </joint>
-  <link name="imu_link"/>
-  <joint name="imu_joint" type="fixed">
-    <parent link="chassis_link"/>
-    <child link="imu_link"/>
-    <origin xyz="0 0 0.15"/>
-  </joint>
-  <link name="camera_link"/>
-  <joint name="camera_joint" type="fixed">
-    <parent link="chassis_link"/>
-    <child link="camera_link"/>
-    <origin xyz="0.25 0 0.35"/>
-  </joint>
-  <link name="gps_link"/>
-  <joint name="gps_joint" type="fixed">
-    <parent link="chassis_link"/>
-    <child link="gps_link"/>
-    <origin xyz="-0.2 0 0.45"/>
-  </joint>
-  <!-- ================= ROS2 CONTROL ================= -->
-  <ros2_control name="ugv_system" type="system">
-    <hardware>
-      <plugin>gazebo_ros2_control/GazeboSystem</plugin>
-    </hardware>
-    <joint name="front_left_wheel_joint">
-      <command_interface name="velocity"/>
-      <state_interface name="position"/>
-      <state_interface name="velocity"/>
-    </joint>
-    <joint name="front_right_wheel_joint">
-      <command_interface name="velocity"/>
-      <state_interface name="position"/>
-      <state_interface name="velocity"/>
-    </joint>
-    <joint name="rear_left_wheel_joint">
-      <command_interface name="velocity"/>
-      <state_interface name="position"/>
-      <state_interface name="velocity"/>
-    </joint>
-    <joint name="rear_right_wheel_joint">
-      <command_interface name="velocity"/>
-      <state_interface name="position"/>
-      <state_interface name="velocity"/>
-    </joint>
-  </ros2_control>
-  <gazebo>
-    <plugin filename="libgazebo_ros2_control.so" name="gazebo_ros2_control">
-      <parameters>$(find rover_simulation)/config/controllers.yaml</parameters>
-    </plugin>
-  </gazebo>
-</robot>
+/home/ugv_dev/ugv_autonomy_stack/ugv_autonomy_stack/src/rover_description/urdf/rover.urdf.xacro

File: src/rover_description/urdf/rover.urdf.xacro (robot description, xacro)
@@ -1,52 +1,43 @@
 <?xml version="1.0"?>
 <robot name="ugv" xmlns:xacro="http://www.ros.org/wiki/xacro">
-  <!-- ================= BASE FRAME (AXLE FRAME) ================= -->
-  <link name="base_link"/>
-  <!-- ================= CHASSIS ================= -->
-  <link name="chassis_link">
+  <!-- ================= BASE FOOTPRINT (ROOT) ================= -->
+  <link name="base_footprint"/>
+  <joint name="base_footprint_joint" type="fixed">
+    <parent link="base_footprint"/>
+    <child link="base_link"/>
+    <origin xyz="0 0 0.2" rpy="0 0 0"/>
+  </joint>
+  <!-- ================= BASE LINK (PHYSICS ROOT) ================= -->
+  <link name="base_link">
     <inertial>
-      <mass value="450.0"/>
-      <origin xyz="0 0 0.2"/>
-      <inertia ixx="60" iyy="42" izz="91.5"
-               ixy="0" ixz="0" iyz="0"/>
+      <mass value="50.0"/>
+      <origin xyz="0 0 0.1"/>
+      <inertia ixx="1.0" ixy="0" ixz="0" iyy="1.0" iyz="0" izz="1.0"/>
     </inertial>
     <visual>
-      <origin xyz="0 0 0.2"/>
-      <geometry>
-        <box size="1.0 1.2 0.4"/>
-      </geometry>
+      <origin xyz="0 0 0.1"/>
+      <geometry><box size="1.0 0.6 0.2"/></geometry>
+      <material name="chassis_color"><color rgba="0.5 0.5 0.5 1.0"/></material>
     </visual>
     <collision>
-      <origin xyz="0 0 0.2"/>
-      <geometry>
-        <box size="1.0 1.2 0.4"/>
-      </geometry>
+      <origin xyz="0 0 0.1"/>
+      <geometry><box size="1.0 0.6 0.2"/></geometry>
     </collision>
   </link>
-  <joint name="base_to_chassis" type="fixed">
-    <parent link="base_link"/>
-    <child link="chassis_link"/>
-    <origin xyz="0 0 -0.092"/>
-  </joint>
   <!-- ================= WHEEL MACRO ================= -->
   <xacro:macro name="wheel" params="name x y">
     <link name="${name}">
       <visual>
-        <origin rpy="1.5707 0 0"/>
-        <geometry>
-          <cylinder radius="0.292" length="0.12"/>
-        </geometry>
+        <origin xyz="0 0 0" rpy="${pi/2} 0 0"/>
+        <geometry><cylinder radius="0.2" length="0.1"/></geometry>
+        <material name="wheel_color"><color rgba="0.1 0.1 0.1 1.0"/></material>
       </visual>
       <collision>
-        <origin rpy="1.5707 0 0"/>
-        <geometry>
-          <cylinder radius="0.292" length="0.12"/>
-        </geometry>
+        <origin xyz="0 0 0" rpy="${pi/2} 0 0"/>
+        <geometry><cylinder radius="0.2" length="0.1"/></geometry>
       </collision>
       <inertial>
-        <mass value="15"/>
-        <origin xyz="0 0 0"/>
-        <inertia ixx="0.34" iyy="0.34" izz="0.64"
-                 ixy="0" ixz="0" iyz="0"/>
+        <mass value="5.0"/>
+        <inertia ixx="0.1" ixy="0" ixz="0" iyy="0.1" iyz="0" izz="0.1"/>
       </inertial>
     </link>
@@ -56,71 +47,106 @@
       <origin xyz="${x} ${y} 0"/>
       <axis xyz="0 1 0"/>
+      <limit effort="1000" velocity="10.0"/>
+      <dynamics damping="0.1" friction="0.1"/>
     </joint>
     <gazebo reference="${name}">
-      <mu1>3.0</mu1>
-      <mu2>3.0</mu2>
-      <kp>100000</kp>
-      <kd>10</kd>
+      <mu1 value="1.0"/>
+      <mu2 value="1.0"/>
+      <kp value="10000000.0"/>
+      <kd value="1.0"/>
+      <material>Gazebo/Grey</material>
     </gazebo>
   </xacro:macro>
   <!-- ================= WHEELS ================= -->
-  <xacro:wheel name="front_left_wheel"  x="0.4"  y="0.675"/>
-  <xacro:wheel name="front_right_wheel" x="0.4"  y="-0.675"/>
-  <xacro:wheel name="rear_left_wheel"   x="-0.4" y="0.675"/>
-  <xacro:wheel name="rear_right_wheel"  x="-0.4" y="-0.675"/>
+  <xacro:wheel name="front_left_wheel"  x="0.4"  y="0.35"/>
+  <xacro:wheel name="front_right_wheel" x="0.4"  y="-0.35"/>
+  <xacro:wheel name="rear_left_wheel"   x="-0.4" y="0.35"/>
+  <xacro:wheel name="rear_right_wheel"  x="-0.4" y="-0.35"/>
   <!-- ================= SENSORS ================= -->
-  <link name="lidar_link"/>
+  <link name="lidar_link">
+    <inertial>
+      <mass value="0.1"/>
+      <origin xyz="0 0 0"/>
+      <inertia ixx="0.001" ixy="0" ixz="0" iyy="0.001" iyz="0" izz="0.001"/>
+    </inertial>
+  </link>
   <joint name="lidar_joint" type="fixed">
-    <parent link="chassis_link"/>
+    <parent link="base_link"/>
     <child link="lidar_link"/>
-    <origin xyz="0.2 0 0.4"/>
+    <origin xyz="0.4 0 0.2"/>
   </joint>
+  <gazebo reference="lidar_link">
+    <sensor name="lidar" type="ray">
+      <visualize>true</visualize>
+      <update_rate>10</update_rate>
+      <ray>
+        <scan>
+          <horizontal>
+            <samples>360</samples>
+            <min_angle>-3.14</min_angle>
+            <max_angle>3.14</max_angle>
+          </horizontal>
+        </scan>
+        <range>
+          <min>0.3</min>
+          <max>12.0</max>
+        </range>
+      </ray>
+      <plugin name="lidar_plugin" filename="libgazebo_ros_ray_sensor.so">
+        <ros>
+          <remapping>~/out:=scan</remapping>
+        </ros>
+        <output_type>sensor_msgs/LaserScan</output_type>
+        <frame_name>lidar_link</frame_name>
+      </plugin>
+    </sensor>
+  </gazebo>
   <link name="imu_link"/>
   <joint name="imu_joint" type="fixed">
-    <parent link="chassis_link"/>
+    <parent link="base_link"/>
     <child link="imu_link"/>
-    <origin xyz="0 0 0.15"/>
+    <origin xyz="0 0 0.1"/>
   </joint>
-  <link name="camera_link"/>
-  <joint name="camera_joint" type="fixed">
-    <parent link="chassis_link"/>
-    <child link="camera_link"/>
-    <origin xyz="0.25 0 0.35"/>
-  </joint>
-  <link name="gps_link"/>
-  <joint name="gps_joint" type="fixed">
-    <parent link="chassis_link"/>
-    <child link="gps_link"/>
-    <origin xyz="-0.2 0 0.45"/>
-  </joint>
-  <!-- ================= ROS2 CONTROL ================= -->
-  <ros2_control name="ugv_system" type="system">
-    <hardware>
-      <plugin>gazebo_ros2_control/GazeboSystem</plugin>
-    </hardware>
-    <joint name="front_left_wheel_joint">
-      <command_interface name="velocity"/>
-      <state_interface name="position"/>
-      <state_interface name="velocity"/>
-    </joint>
-    <joint name="front_right_wheel_joint">
-      <command_interface name="velocity"/>
-      <state_interface name="position"/>
-      <state_interface name="velocity"/>
-    </joint>
-    <joint name="rear_left_wheel_joint">
-      <command_interface name="velocity"/>
-      <state_interface name="position"/>
-      <state_interface name="velocity"/>
-    </joint>
-    <joint name="rear_right_wheel_joint">
-      <command_interface name="velocity"/>
-      <state_interface name="position"/>
-      <state_interface name="velocity"/>
-    </joint>
-  </ros2_control>
+  <gazebo reference="imu_link">
+    <sensor name="imu_sensor" type="imu">
+      <plugin name="imu_plugin" filename="libgazebo_ros_imu_sensor.so">
+        <ros>
+          <remapping>~/out:=imu</remapping>
+        </ros>
+      </plugin>
+    </sensor>
+  </gazebo>
+  <!-- ================= DIRECT GAZEBO MOBILITY (PROXY) ================= -->
   <gazebo>
-    <plugin filename="libgazebo_ros2_control.so" name="gazebo_ros2_control">
-      <parameters>$(find rover_simulation)/config/controllers.yaml</parameters>
+    <plugin name="diff_drive" filename="libgazebo_ros_diff_drive.so">
+      <ros>
+        <namespace>/</namespace>
+        <remapping>cmd_vel:=diff_drive_controller/cmd_vel_unstamped</remapping>
+        <remapping>odom:=diff_drive_controller/odom</remapping>
+      </ros>
+      <num_wheel_pairs>2</num_wheel_pairs>
+      <left_joint>front_left_wheel_joint</left_joint>
+      <left_joint>rear_left_wheel_joint</left_joint>
+      <right_joint>front_right_wheel_joint</right_joint>
+      <right_joint>rear_right_wheel_joint</right_joint>
+      <wheel_separation>0.7</wheel_separation>
+      <wheel_diameter>0.4</wheel_diameter>
+      <max_wheel_torque>200</max_wheel_torque>
+      <max_wheel_acceleration>5.0</max_wheel_acceleration>
+      <publish_odom>true</publish_odom>
+      <publish_odom_tf>true</publish_odom_tf>
+      <publish_wheel_tf>true</publish_wheel_tf>
+      <odometry_frame>odom</odometry_frame>
+      <robot_base_frame>base_footprint</robot_base_frame>
+    </plugin>
+    <plugin name="joint_state_publisher" filename="libgazebo_ros_joint_state_publisher.so">
+      <ros>
+        <remapping>joint_states:=joint_states</remapping>
+      </ros>
+      <update_rate>50</update_rate>
+      <joint_name>front_left_wheel_joint</joint_name>
+      <joint_name>front_right_wheel_joint</joint_name>
+      <joint_name>rear_left_wheel_joint</joint_name>
+      <joint_name>rear_right_wheel_joint</joint_name>
     </plugin>
   </gazebo>
